Commit message: start rosie with arms tucked using tuck_presim script, and waiting for "simulation started" message

File: rosie/baxter_base.urdf.xacro (robot description, xacro)
@@ -153,5 +153,5 @@
       <origin rpy="0 0 0.0" xyz="-0.07 -0.04 0.0"/>
       <geometry>
-        <sphere radius="0.22"/>
+        <sphere radius="0.08"/>
       </geometry>
     </collision>
@@ -175,5 +175,5 @@
       <origin rpy="0 0 0" xyz="-0.07 0.04 0.00"/>
       <geometry>
-        <sphere radius="0.22"/>
+        <sphere radius="0.08"/>
       </geometry>
     </collision>
@@ -533,5 +533,5 @@
     <parent link="right_lower_shoulder"/>
     <child link="right_upper_elbow"/>
-    <limit effort="50.0" lower="-3.05417993878" upper="3.05417993878" velocity="1.5"/>
+    <limit effort="50.0" lower="-3.25417993878" upper="3.25417993878" velocity="1.5"/>
     <dynamics damping="0.7" friction="0.0"/>
   </joint>
@@ -901,5 +901,5 @@
     <parent link="left_lower_shoulder"/>
     <child link="left_upper_elbow"/>
-    <limit effort="50.0" lower="-3.05417993878" upper="3.05417993878" velocity="1.5"/>
+    <limit effort="50.0" lower="-3.25417993878" upper="3.25417993878" velocity="1.5"/>
     <dynamics damping="0.7" friction="0.0"/>
   </joint>
