Commit message: Added sensor, added moving actor

File: blue-sim/mir_description/urdf/include/mir_100_v1.urdf.xacro (robot description, xacro)
@@ -193,4 +193,9 @@
     </joint>
     <link name="${prefix}us_2_frame" />
+    <!-- Realsense Sensor -->
+    <xacro:include filename="$(find realsense_gazebo_plugin)/urdf/realsense-RS200.macro.xacro"/>
+    <xacro:realsense-rs200 prefix="${prefix}" parent="base_link">
+      <origin xyz="0 0 0.4" rpy="0 0 0" />
+    </xacro:realsense-rs200>
     <!-- wheels -->
     <xacro:actuated_wheel prefix="${prefix}" locationprefix="left" locationright="-1"/>

Commit message: Sensor debugged, passed topic to human detector, built actor plugin, added code to blue_delivery

File: blue-sim/mir_description/urdf/include/mir_100_v1.urdf.xacro (robot description, xacro)
@@ -196,5 +196,5 @@
     <xacro:include filename="$(find realsense_gazebo_plugin)/urdf/realsense-RS200.macro.xacro"/>
     <xacro:realsense-rs200 prefix="${prefix}" parent="base_link">
-      <origin xyz="0 0 0.4" rpy="0 0 0" />
+      <origin xyz="0.4 0 0.4" rpy="0 0 0" />
     </xacro:realsense-rs200>
     <!-- wheels -->
